File: hmacs_v0.2.kicad_sch (KiCad schematic)
At the start: 12 parts

Commit message: Final changes before first manufacturing run
Parts:
- J1: value (none) -> EXT_CONNECTOR
- J2: value (none) -> MODULE_CONN_2; footprint (none) -> Connector_PinSocket_2.54mm:PinSocket_1x10_P2.54mm_Vertical
- J3: value (none) -> SENSE_PIN_CONNECTOR; footprint (none) -> Connector_PinHeader_2.54mm:PinHeader_1x02_P2.54mm_Vertical
- J4: value (none) -> MODULE_CONN_1; footprint (none) -> Connector_PinSocket_2.54mm:PinSocket_1x16_P2.54mm_Vertical
- J5: value (none) -> AC_INPUT; footprint (none) -> kf301-2p:HANDSON_KF301-2P
- J6: value (none) -> RFID_HEADER; footprint (none) -> Connector_PinSocket_2.54mm:PinSocket_1x08_P2.54mm_Vertical
- J7: value (none) -> RELAY_CONNECTOR; footprint (none) -> Connector_PinHeader_2.54mm:PinHeader_1x03_P2.54mm_Vertical
- J8: value (none) -> SSR_CONNECTOR; footprint (none) -> Connector_PinHeader_2.54mm:PinHeader_1x02_P2.54mm_Vertical
- PS1: value (none) -> HLK-PM01; footprint (none) -> Converter_ACDC:Converter_ACDC_HiLink_HLK-PMxx
- Q1: value (none) -> RELAY_SIG_PNP_EBC; footprint (none) -> Package_TO_SOT_THT:TO-92
- R1: value (none) -> R; footprint (none) -> Resistor_THT:R_Axial_DIN0204_L3.6mm_D1.6mm_P7.62mm_Horizontal
- R2: footprint (none) -> Resistor_THT:R_Axial_DIN0204_L3.6mm_D1.6mm_P7.62mm_Horizontal

Commit message: Fix board errors and bump version to 0.3.0
Parts:
- Q1: value RELAY_SIG_PNP_EBC -> 2N3906; footprint Package_TO_SOT_THT:TO-92 -> Package_TO_SOT_THT:TO-92_Inline; symbol Device:Q_PNP_EBC -> Transistor_BJT:2N3906
Connections:
- net SSR is gone; now on net RELAY: J8.2 (Pin_2), Q1.3 (C), R2.1
- net +3V3: now also Q1.1 (E)
- net +5V: no longer Q1.1 (E)
- net RELAY: no longer J4.6 (Pin_6), R1.1
- new net RELAY_SIG: J4.6 (Pin_6), R1.1
Changed lines of the file:
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@@
     )
   )
-  (global_label "RELAY" (shape input) (at 78.74 80.01 270) (fields_autoplaced)
+  (global_label "RELAY_SIG" (shape input) (at 78.74 80.01 270) (fields_autoplaced)
     (effects (font (size 1.27 1.27)) (justify right))
     (property "Intersheet References" "${INTERSHEET_REFS}" (id 0) (at 78.6606 88.0474 90)
@@
     )
   )
-  (global_label "SSR" (shape input) (at 184.15 110.49 0) (fields_autoplaced)
+  (global_label "RELAY" (shape input) (at 184.15 110.49 0) (fields_autoplaced)
     (effects (font (size 1.27 1.27)) (justify left))
     (property "Intersheet References" "${INTERSHEET_REFS}" (id 0) (at 190.2521 110.4106 0)
@@
     )
   )
-  (global_label "SSR" (shape input) (at 147.32 100.33 0) (fields_autoplaced)
+  (global_label "RELAY" (shape input) (at 147.32 100.33 0) (fields_autoplaced)
     (effects (font (size 1.27 1.27)) (justify left))
     (property "Intersheet References" "${INTERSHEET_REFS}" (id 0) (at 153.4221 100.2506 0)
@@
     )
   )
-  (global_label "RELAY" (shape input) (at 129.54 106.68 180) (fields_autoplaced)
+  (global_label "RELAY_SIG" (shape input) (at 129.54 106.68 180) (fields_autoplaced)
     (effects (font (size 1.27 1.27)) (justify right))
     (property "Intersheet References" "${INTERSHEET_REFS}" (id 0) (at 121.5026 106.6006 0)
@@
     (pin "1")
   )
+  (symbol (lib_id "power:+3.3V") (at 144.78 111.76 180) (unit 1)
+    (in_bom yes) (on_board yes) (fields_autoplaced)
+    (property "Reference" "#PWR0101" (id 0) (at 144.78 107.95 0)
+      (effects (font (size 1.27 1.27)) hide)
+    )
+    (property "Value" "+3.3V" (id 1) (at 144.78 116.2034 0))
+    (property "Footprint" "" (id 2) (at 144.78 111.76 0)
+      (effects (font (size 1.27 1.27)) hide)
+    )
+    (property "Datasheet" "" (id 3) (at 144.78 111.76 0)
+      (effects (font (size 1.27 1.27)) hide)
+    )
+    (pin "1")
+  )
   (symbol (lib_id "power:+5V") (at 184.15 124.46 270) (unit 1)
     (in_bom yes) (on_board yes) (fields_autoplaced)
@@
     )
     (property "Datasheet" "" (id 3) (at 184.15 107.95 0)
-      (effects (font (size 1.27 1.27)) hide)
-    )
-    (pin "1")
-  )
-  (symbol (lib_id "power:+5V") (at 144.78 111.76 180) (unit 1)
-    (in_bom yes) (on_board yes) (fields_autoplaced)
-    (property "Reference" "#PWR018" (id 0) (at 144.78 107.95 0)
-      (effects (font (size 1.27 1.27)) hide)
-    )
-    (property "Value" "+5V" (id 1) (at 144.78 116.2034 0))
-    (property "Footprint" "" (id 2) (at 144.78 111.76 0)
-      (effects (font (size 1.27 1.27)) hide)
-    )
-    (property "Datasheet" "" (id 3) (at 144.78 111.76 0)
       (effects (font (size 1.27 1.27)) hide)
     )
@@
     (pin "2")
   )
-  (symbol (lib_id "Device:Q_PNP_EBC") (at 142.24 106.68 0) (unit 1)
+  (symbol (lib_id "Transistor_BJT:2N3906") (at 142.24 106.68 0) (unit 1)
     (in_bom yes) (on_board yes) (fields_autoplaced)
     (property "Reference" "Q1" (id 0) (at 147.0914 105.8453 0)
       (effects (font (size 1.27 1.27)) (justify left))
     )
-    (property "Value" "RELAY_SIG_PNP_EBC" (id 1) (at 147.0914 108.3822 0)
-      (effects (font (size 1.27 1.27)) (justify left))
-    )
-    (property "Footprint" "Package_TO_SOT_THT:TO-92" (id 2) (at 147.32 104.14 0)
-      (effects (font (size 1.27 1.27)) hide)
-    )
-    (property "Datasheet" "~" (id 3) (at 142.24 106.68 0)
-      (effects (font (size 1.27 1.27)) hide)
+    (property "Value" "2N3906" (id 1) (at 147.0914 108.3822 0)
+      (effects (font (size 1.27 1.27)) (justify left))
+    )
+    (property "Footprint" "Package_TO_SOT_THT:TO-92_Inline" (id 2) (at 147.32 108.585 0)
+      (effects (font (size 1.27 1.27) italic) (justify left) hide)
+    )
+    (property "Datasheet" "https://www.onsemi.com/pub/Collateral/2N3906-D.PDF" (id 3) (at 142.24 106.68 0)
+      (effects (font (size 1.27 1.27)) (justify left) hide)
     )
     (pin "1")
@@
       (reference "#PWR017") (unit 1) (value "GND") (footprint "")
     )
-    (path "/b68d9dfa-6ef2-44f0-823b-4595e7055939"
-      (reference "#PWR018") (unit 1) (value "+5V") (footprint "")
-    )
     (path "/4b31a572-7057-4b3b-ad00-5a5d597e8042"
       (reference "#PWR019") (unit 1) (value "+5V") (footprint "")
@@
       (reference "#PWR021") (unit 1) (value "GND") (footprint "")
     )
+    (path "/3706cd11-0019-4e23-b082-f2bfc5537019"
+      (reference "#PWR0101") (unit 1) (value "+3.3V") (footprint "")
+    )
     (path "/b584827c-9416-48d9-9c16-1f4af2b091f1"
       (reference "J1") (unit 1) (value "EXT_CONNECTOR") (footprint "Connector_PinHeader_2.54mm:PinHeader_1x03_P2.54mm_Vertical")
@@
     )
     (path "/f90fbac7-ec48-4a76-a2ed-0a8a9e837154"
-      (reference "Q1") (unit 1) (value "RELAY_SIG_PNP_EBC") (footprint "Package_TO_SOT_THT:TO-92")
+      (reference "Q1") (unit 1) (value "2N3906") (footprint "Package_TO_SOT_THT:TO-92_Inline")
     )
     (path "/1493b2a1-5d15-4a3f-8f99-6617bf4184b6"
